File: hardware/HeadphoneAmp/PowerSupplies.kicad_sch (KiCad schematic)
At the start: 22 parts, among them J10 Barrel_Jack_Switch, J11 Router Power, U10 MIC5317, U7 L7812ACV, U8 L7912ACV, U9 MCP1755ST-5002xDB

Commit message: Switched a pile of footprints over to our own versions
Parts:
- C13, C14: footprint Capacitor_THT:CP_Radial_D10.0mm_P5.00mm -> rhais_rcl:CP_Radial_D10.0mm_P5.00mm
- C15, C16: footprint Capacitor_THT:CP_Radial_D8.0mm_P3.50mm -> rhais_rcl:CP_Radial_D8.0mm_P3.50mm
- D1, D2: footprint Diode_SMD:D_SMA -> rhais_diode:D_SMA
- J10: footprint Connector_BarrelJack:BarrelJack_GCT_DCJ200-10-A_Horizontal -> rhais_connector-jack:BarrelJack_GCT_DCJ200-10-A_Horizontal
- J11: footprint Connector_PinHeader_2.54mm:PinHeader_1x01_P2.54mm_Vertical -> rhais_connector-pinheader:PinHeader_1x01_P2.54mm_Vertical
- U7, U8: footprint Package_TO_SOT_THT:TO-220-3_Vertical -> rhais_package-to:TO-220-3_Vertical
Changed lines of the file:
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@@
     (property "Reference" "D1" (id 0) (at 58.42 88.9 0))
     (property "Value" "B160-13-F" (id 1) (at 58.42 93.98 0))
-    (property "Footprint" "Diode_SMD:D_SMA" (id 2) (at 58.42 91.44 90)
+    (property "Footprint" "rhais_diode:D_SMA" (id 2) (at 58.42 91.44 90)
       (effects (font (size 1.27 1.27)) hide)
     )
@@
     (property "Reference" "C14" (id 0) (at 60.96 106.68 90))
     (property "Value" "680u" (id 1) (at 66.04 106.68 90))
-    (property "Footprint" "Capacitor_THT:CP_Radial_D10.0mm_P5.00mm" (id 2) (at 63.5 106.68 0)
+    (property "Footprint" "rhais_rcl:CP_Radial_D10.0mm_P5.00mm" (id 2) (at 63.5 106.68 0)
       (effects (font (size 1.27 1.27)) hide)
     )
@@
     (property "Reference" "J10" (id 0) (at 40.64 96.266 0))
     (property "Value" "Barrel_Jack_Switch" (id 1) (at 40.64 106.68 0))
-    (property "Footprint" "Connector_BarrelJack:BarrelJack_GCT_DCJ200-10-A_Horizontal" (id 2) (at 41.91 102.616 0)
+    (property "Footprint" "rhais_connector-jack:BarrelJack_GCT_DCJ200-10-A_Horizontal" (id 2) (at 41.91 102.616 0)
       (effects (font (size 1.27 1.27)) hide)
     )
@@
     (property "Reference" "C16" (id 0) (at 68.58 106.68 90))
     (property "Value" "330u" (id 1) (at 73.66 106.68 90))
-    (property "Footprint" "Capacitor_THT:CP_Radial_D8.0mm_P3.50mm" (id 2) (at 71.12 106.68 0)
+    (property "Footprint" "rhais_rcl:CP_Radial_D8.0mm_P3.50mm" (id 2) (at 71.12 106.68 0)
       (effects (font (size 1.27 1.27)) hide)
     )
@@
     (property "Reference" "C15" (id 0) (at 68.58 96.52 90))
     (property "Value" "330u" (id 1) (at 73.66 96.52 90))
-    (property "Footprint" "Capacitor_THT:CP_Radial_D8.0mm_P3.50mm" (id 2) (at 71.12 96.52 0)
+    (property "Footprint" "rhais_rcl:CP_Radial_D8.0mm_P3.50mm" (id 2) (at 71.12 96.52 0)
       (effects (font (size 1.27 1.27)) hide)
     )
@@
     (property "Reference" "D2" (id 0) (at 58.42 109.22 0))
     (property "Value" "B160-13-F" (id 1) (at 58.42 114.3 0))
-    (property "Footprint" "Diode_SMD:D_SMA" (id 2) (at 58.42 111.76 90)
+    (property "Footprint" "rhais_diode:D_SMA" (id 2) (at 58.42 111.76 90)
       (effects (font (size 1.27 1.27)) hide)
     )
@@
     )
     (property "Value" "L7912ACV" (id 1) (at 88.9 114.935 0))
-    (property "Footprint" "Package_TO_SOT_THT:TO-220-3_Vertical" (id 2) (at 88.9 116.84 0)
+    (property "Footprint" "rhais_package-to:TO-220-3_Vertical" (id 2) (at 88.9 116.84 0)
       (effects (font (size 1.27 1.27) italic) hide)
     )
@@
     (property "Reference" "C13" (id 0) (at 60.96 96.52 90))
     (property "Value" "680u" (id 1) (at 66.04 96.52 90))
-    (property "Footprint" "Capacitor_THT:CP_Radial_D10.0mm_P5.00mm" (id 2) (at 63.5 96.52 0)
+    (property "Footprint" "rhais_rcl:CP_Radial_D10.0mm_P5.00mm" (id 2) (at 63.5 96.52 0)
       (effects (font (size 1.27 1.27)) hide)
     )
@@
     (property "Reference" "J11" (id 0) (at 109.22 96.52 0))
     (property "Value" "Router Power" (id 1) (at 104.14 92.71 0))
-    (property "Footprint" "Connector_PinHeader_2.54mm:PinHeader_1x01_P2.54mm_Vertical" (id 2) (at 106.68 96.52 0)
+    (property "Footprint" "rhais_connector-pinheader:PinHeader_1x01_P2.54mm_Vertical" (id 2) (at 106.68 96.52 0)
       (effects (font (size 1.27 1.27)) hide)
     )
@@
     )
     (property "Value" "L7812ACV" (id 1) (at 88.9 88.265 0))
-    (property "Footprint" "Package_TO_SOT_THT:TO-220-3_Vertical" (id 2) (at 89.535 95.25 0)
+    (property "Footprint" "rhais_package-to:TO-220-3_Vertical" (id 2) (at 89.535 95.25 0)
       (effects (font (size 1.27 1.27) italic) (justify left) hide)
     )
