File: hardware/HeadphoneAmp/DigitalInterface.kicad_sch (KiCad schematic)
At the start: 23 parts, among them U11 PCM1796DB, U12 ACPL-064L, U13 ACPL-064L, U14 APS1551SZ, U15 ACPL-064L, U16 ACPL-M61L

Commit message: Cleanup in the base board
Other:
- note removed: "❯ icepll -b -o 33.8688 F_PLLIN: 11.059 MHz (given) F_PLLOUT: 33.869 MHz (requested) F_PLLOUT: 33.869 MHz (achieved) FEEDBACK: SIMPLE F_PFD: 11.059 MHz F_VCO: 541.901 MHz DIVR: 0 (4'b0000) DIVF: 48 (7'b0110000) DIVQ: 4 (3'b100) FILTER_RANGE: 1 (3'b001)"
- note removed: "❯ icepll -i 24.576 -o 36.864 F_PLLIN: 24.576 MHz (given) F_PLLOUT: 36.864 MHz (requested) F_PLLOUT: 36.864 MHz (achieved) FEEDBACK: SIMPLE F_PFD: 24.576 MHz F_VCO: 589.824 MHz DIVR: 0 (4'b0000) DIVF: 23 (7'b0010111) DIVQ: 4 (3'b100) FILTER_RANGE: 2 (3'b010)"
Changed lines of the file:
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@@
     (stroke (width 0) (type default) (color 0 0 0 0))
-  )
-  (text "❯ icepll -i 24.576 -o 36.864\n\nF_PLLIN:    24.576 MHz (given)\nF_PLLOUT:   36.864 MHz (requested)\nF_PLLOUT:   36.864 MHz (achieved)\n\nFEEDBACK: SIMPLE\nF_PFD:   24.576 MHz\nF_VCO:  589.824 MHz\n\nDIVR:  0 (4'b0000)\nDIVF: 23 (7'b0010111)\nDIVQ:  4 (3'b100)\n\nFILTER_RANGE: 2 (3'b010)\n"
-    (at 127 190.5 0)
-    (effects (font (size 1.27 1.27)) (justify left bottom))
   )
   (text "SYS_CLK must be one of\n24.576MHz (32kHz)\n33.8688MHz (44k1Hz)\n36.864MHz (48kHz+)\ndepending on sampling frequency"
@@
     (effects (font (size 1.27 1.27)) (justify right bottom))
   )
-  (text "❯ icepll -b -o 33.8688\n\nF_PLLIN:    11.059 MHz (given)\nF_PLLOUT:   33.869 MHz (requested)\nF_PLLOUT:   33.869 MHz (achieved)\n\nFEEDBACK: SIMPLE\nF_PFD:   11.059 MHz\nF_VCO:  541.901 MHz\n\nDIVR:  0 (4'b0000)\nDIVF: 48 (7'b0110000)\nDIVQ:  4 (3'b100)\n\nFILTER_RANGE: 1 (3'b001)"
-    (at 88.9 190.5 0)
-    (effects (font (size 1.27 1.27)) (justify left bottom))
-  )
   (text "~{RST} is only needed if we\nwant to manually reset the\nchip, but if we're smart with\nSPI, this is unnecessary"

Commit message: Completed a pile more work on the various boards that comprise the project
Parts:
- H3, H4: now left out of the parts list
Changed lines of the file:
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@@
   )
   (symbol (lib_id "Mechanical:MountingHole_Pad") (at 58.42 165.1 90) (unit 1)
-    (in_bom yes) (on_board yes)
+    (in_bom no) (on_board yes)
     (property "Reference" "H3" (id 0) (at 54.61 165.1 90)
       (effects (font (size 1.27 1.27)) (justify left))
@@
   )
   (symbol (lib_id "Mechanical:MountingHole_Pad") (at 68.58 165.1 270) (unit 1)
-    (in_bom yes) (on_board yes)
+    (in_bom no) (on_board yes)
     (property "Reference" "H4" (id 0) (at 72.39 165.1 90)
       (effects (font (size 1.27 1.27)) (justify left))
