File: hardware/HeadphoneAmp/HeadphoneAmp.kicad_pcb (KiCad board)
At the start: 4 copper layers, 100 x 80 mm, 134 parts, among them J1 Preamp Input, J10 Barrel_Jack_Switch, J11 Router Power, J2 Source, J3 1503_02, J4 1503_02, J5 In R, J6 In L, J7 I2S + SPI, J8 Out R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

Commit message: Made the headphone amp + DAC board's refdes fabulous
Parts:
- D1, D2: value SS16 -> B160-13-F
- J1: footprint Connector_PinHeader_2.54mm:PinHeader_1x03_P2.54mm_Vertical -> rhais_connector-pinheader:PinHeader_1x03_P2.54mm_Vertical
- moved J1 2.54 mm to (128.0, 122.5)

Commit message: Switched a pile of footprints over to our own versions
Parts:
- C13, C14: footprint Capacitor_THT:CP_Radial_D10.0mm_P5.00mm -> rhais_rcl:CP_Radial_D10.0mm_P5.00mm
- C15, C16: footprint Capacitor_THT:CP_Radial_D8.0mm_P3.50mm -> rhais_rcl:CP_Radial_D8.0mm_P3.50mm
- D1, D2: footprint Diode_SMD:D_SMA -> rhais_diode:D_SMA
- J10: footprint Connector_BarrelJack:BarrelJack_GCT_DCJ200-10-A_Horizontal -> rhais_connector-jack:BarrelJack_GCT_DCJ200-10-A_Horizontal
- J11, J2: footprint Connector_PinHeader_2.54mm:PinHeader_1x01_P2.54mm_Vertical -> rhais_connector-pinheader:PinHeader_1x01_P2.54mm_Vertical
- U7, U8: footprint Package_TO_SOT_THT:TO-220-3_Vertical -> rhais_package-to:TO-220-3_Vertical
- moved U7 2.54 mm to (154.0, 102.0)
- moved U8 2.54 mm to (142.0, 102.0)
- moved C13 2.50 mm to (154.5, 112.0)
- moved C14 2.50 mm to (146.5, 120.5)
- moved C15 1.75 mm to (156.0, 121.5)
- moved C16 1.75 mm to (145.0, 111.0)

Commit message: Cleanup in the base board
Other:
- outline, holes or cut-outs redrawn
Changed lines of the file:
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@@
   (gr_arc (start 186 100.5) (mid 186.8 101.3) (end 186 102.1) (layer "Edge.Cuts") (width 0.05))
   (gr_arc locked (start 100.5 140) (mid 100.146447 139.853553) (end 100 139.5) (layer "Edge.Cuts") (width 0.05))
-  (gr_line locked (start 130 140) (end 174 140) (layer "Edge.Cuts") (width 0.05))
+  (gr_line locked (start 130 140) (end 173.5 140) (layer "Edge.Cuts") (width 0.05))
   (gr_arc locked (start 200 139.5) (mid 199.853553 139.853553) (end 199.5 140) (layer "Edge.Cuts") (width 0.05))
   (gr_line locked (start 100.5 60) (end 126 60) (layer "Edge.Cuts") (width 0.05))
-  (gr_line locked (start 192 140) (end 192 134) (layer "Edge.Cuts") (width 0.05))
-  (gr_line locked (start 199.5 140) (end 192 140) (layer "Edge.Cuts") (width 0.05))
+  (gr_arc locked (start 192.5 140) (mid 192.146447 139.853553) (end 192 139.5) (layer "Edge.Cuts") (width 0.05))
+  (gr_line locked (start 192 139.5) (end 192 134.5) (layer "Edge.Cuts") (width 0.05))
+  (gr_line locked (start 199.5 140) (end 192.5 140) (layer "Edge.Cuts") (width 0.05))
   (gr_line (start 172 100.5) (end 186 100.5) (layer "Edge.Cuts") (width 0.05))
+  (gr_arc locked (start 191.5 134) (mid 191.853553 134.146447) (end 192 134.5) (layer "Edge.Cuts") (width 0.05))
+  (gr_arc locked (start 174 134.5) (mid 174.146447 134.146447) (end 174.5 134) (layer "Edge.Cuts") (width 0.05))
   (gr_arc locked (start 100 60.5) (mid 100.146447 60.146447) (end 100.5 60) (layer "Edge.Cuts") (width 0.05))
   (gr_arc (start 172 102.1) (mid 171.2 101.3) (end 172 100.5) (layer "Edge.Cuts") (width 0.05))
   (gr_line locked (start 100 139.5) (end 100 60.5) (layer "Edge.Cuts") (width 0.05))
   (gr_line locked (start 200 139.5) (end 200 60.5) (layer "Edge.Cuts") (width 0.05))
-  (gr_line locked (start 174 134) (end 174 140) (layer "Edge.Cuts") (width 0.05))
+  (gr_line locked (start 174 134.5) (end 174 139.5) (layer "Edge.Cuts") (width 0.05))
   (gr_arc locked (start 199.5 60) (mid 199.853553 60.146447) (end 200 60.5) (layer "Edge.Cuts") (width 0.05))
+  (gr_arc locked (start 174 139.5) (mid 173.853553 139.853553) (end 173.5 140) (layer "Edge.Cuts") (width 0.05))
   (gr_line locked (start 100.5 140) (end 126 140) (layer "Edge.Cuts") (width 0.05))
   (gr_line (start 186 102.1) (end 172 102.1) (layer "Edge.Cuts") (width 0.05))
-  (gr_line locked (start 174 134) (end 192 134) (layer "Edge.Cuts") (width 0.05))
+  (gr_line locked (start 174.5 134) (end 191.5 134) (layer "Edge.Cuts") (width 0.05))
   (gr_line locked (start 130 60) (end 199.5 60) (layer "Edge.Cuts") (width 0.05))
   (gr_text "v2 Strict" (at 113.9 115.8) (layer "F.SilkS")
