File: hardware/HeadphoneAmp/HeadphoneAmp.kicad_sch (KiCad schematic)
At the start: 29 parts, among them J1 Preamp Input, J2 Source, J3 1503_02, J4 1503_02, J5 In R, J6 In L, J7 I2S + SPI, J8 Out R, J9 Out L, SW1 SW_SPDT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

Commit message: Switched a couple of footprints, cleaning up the amp+dac board
Parts:
- J1: footprint Connector_PinHeader_2.54mm:PinHeader_1x03_P2.54mm_Vertical -> rhais_connector-pinheader:PinHeader_1x03_P2.54mm_Vertical
Changed lines of the file:
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@@
     (property "Reference" "J1" (id 0) (at 38.1 71.12 0))
     (property "Value" "Preamp Input" (id 1) (at 35.56 76.2 90))
-    (property "Footprint" "Connector_PinHeader_2.54mm:PinHeader_1x03_P2.54mm_Vertical" (id 2) (at 38.1 76.2 0)
+    (property "Footprint" "rhais_connector-pinheader:PinHeader_1x03_P2.54mm_Vertical" (id 2) (at 38.1 76.2 0)
       (effects (font (size 1.27 1.27)) hide)
     )
@@
     )
     (path "/ad1c7d30-fa47-47fd-bb07-e836ca23dcc6"
-      (reference "J1") (unit 1) (value "Preamp Input") (footprint "Connector_PinHeader_2.54mm:PinHeader_1x03_P2.54mm_Vertical")
+      (reference "J1") (unit 1) (value "Preamp Input") (footprint "rhais_connector-pinheader:PinHeader_1x03_P2.54mm_Vertical")
     )
     (path "/24b3bc61-d595-4851-a8f5-193039965902"

Commit message: Switched a pile of footprints over to our own versions
Parts:
- J2: footprint Connector_PinHeader_2.54mm:PinHeader_1x01_P2.54mm_Vertical -> rhais_connector-pinheader:PinHeader_1x01_P2.54mm_Vertical
Changed lines of the file:
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@@
     (property "Reference" "J2" (id 0) (at 60.96 22.86 0))
     (property "Value" "Source" (id 1) (at 60.96 27.94 0))
-    (property "Footprint" "Connector_PinHeader_2.54mm:PinHeader_1x01_P2.54mm_Vertical" (id 2) (at 60.96 25.4 0)
+    (property "Footprint" "rhais_connector-pinheader:PinHeader_1x01_P2.54mm_Vertical" (id 2) (at 60.96 25.4 0)
       (effects (font (size 1.27 1.27)) hide)
     )
@@
     )
     (path "/090c9c05-427a-444a-8689-526c4a2a5969/d376684b-c98b-4996-a53e-16c44de4793c"
-      (reference "C13") (unit 1) (value "680u") (footprint "Capacitor_THT:CP_Radial_D10.0mm_P5.00mm")
+      (reference "C13") (unit 1) (value "680u") (footprint "rhais_rcl:CP_Radial_D10.0mm_P5.00mm")
     )
     (path "/090c9c05-427a-444a-8689-526c4a2a5969/2500a677-af13-47ef-af71-92d4c6b9af26"
-      (reference "C14") (unit 1) (value "680u") (footprint "Capacitor_THT:CP_Radial_D10.0mm_P5.00mm")
+      (reference "C14") (unit 1) (value "680u") (footprint "rhais_rcl:CP_Radial_D10.0mm_P5.00mm")
     )
     (path "/090c9c05-427a-444a-8689-526c4a2a5969/88bcbb96-1352-4e82-adab-44016974caa4"
-      (reference "C15") (unit 1) (value "330u") (footprint "Capacitor_THT:CP_Radial_D8.0mm_P3.50mm")
+      (reference "C15") (unit 1) (value "330u") (footprint "rhais_rcl:CP_Radial_D8.0mm_P3.50mm")
     )
     (path "/090c9c05-427a-444a-8689-526c4a2a5969/70278fec-9fb2-4c5d-8718-ad8b10962001"
-      (reference "C16") (unit 1) (value "330u") (footprint "Capacitor_THT:CP_Radial_D8.0mm_P3.50mm")
+      (reference "C16") (unit 1) (value "330u") (footprint "rhais_rcl:CP_Radial_D8.0mm_P3.50mm")
     )
     (path "/090c9c05-427a-444a-8689-526c4a2a5969/28aaba3d-12b6-418b-a744-2c9be55de702"
@@
     )
     (path "/090c9c05-427a-444a-8689-526c4a2a5969/06911b3c-ed0a-4e2d-88a7-7f4be8891733"
-      (reference "D1") (unit 1) (value "B160-13-F") (footprint "Diode_SMD:D_SMA")
+      (reference "D1") (unit 1) (value "B160-13-F") (footprint "rhais_diode:D_SMA")
     )
     (path "/090c9c05-427a-444a-8689-526c4a2a5969/8c5a408b-1fa2-4c32-aba4-7aa1052abd18"
-      (reference "D2") (unit 1) (value "B160-13-F") (footprint "Diode_SMD:D_SMA")
+      (reference "D2") (unit 1) (value "B160-13-F") (footprint "rhais_diode:D_SMA")
     )
     (path "/58956b23-7a9e-4cb8-a8aa-a3b38807c559"
@@
     )
     (path "/24b3bc61-d595-4851-a8f5-193039965902"
-      (reference "J2") (unit 1) (value "Source") (footprint "Connector_PinHeader_2.54mm:PinHeader_1x01_P2.54mm_Vertical")
+      (reference "J2") (unit 1) (value "Source") (footprint "rhais_connector-pinheader:PinHeader_1x01_P2.54mm_Vertical")
     )
     (path "/39e48209-95b8-454d-a3ad-2994fb8b8c0a"
@@
     )
     (path "/090c9c05-427a-444a-8689-526c4a2a5969/4b2c7b21-888f-49ea-8818-782e678821c4"
-      (reference "J10") (unit 1) (value "Barrel_Jack_Switch") (footprint "Connector_BarrelJack:BarrelJack_GCT_DCJ200-10-A_Horizontal")
+      (reference "J10") (unit 1) (value "Barrel_Jack_Switch") (footprint "rhais_connector-jack:BarrelJack_GCT_DCJ200-10-A_Horizontal")
     )
     (path "/090c9c05-427a-444a-8689-526c4a2a5969/dd810f41-bbfe-43b8-8214-aa818844392c"
-      (reference "J11") (unit 1) (value "Router Power") (footprint "Connector_PinHeader_2.54mm:PinHeader_1x01_P2.54mm_Vertical")
+      (reference "J11") (unit 1) (value "Router Power") (footprint "rhais_connector-pinheader:PinHeader_1x01_P2.54mm_Vertical")
     )
     (path "/83f821ce-fe44-4600-b473-90e23f79c6dc/f4d33b1b-105b-40d7-ae29-0a0c74ed0cf4"
@@
     )
     (path "/090c9c05-427a-444a-8689-526c4a2a5969/f9ff6624-58ac-4f2a-8494-ba0471b48006"
-      (reference "U7") (unit 1) (value "L7812ACV") (footprint "Package_TO_SOT_THT:TO-220-3_Vertical")
+      (reference "U7") (unit 1) (value "L7812ACV") (footprint "rhais_package-to:TO-220-3_Vertical")
     )
     (path "/090c9c05-427a-444a-8689-526c4a2a5969/b43f46da-c122-4689-8cf0-8d7c66a60c5b"
-      (reference "U8") (unit 1) (value "L7912ACV") (footprint "Package_TO_SOT_THT:TO-220-3_Vertical")
+      (reference "U8") (unit 1) (value "L7912ACV") (footprint "rhais_package-to:TO-220-3_Vertical")
     )
     (path "/090c9c05-427a-444a-8689-526c4a2a5969/d1320b24-3b97-4732-bb23-3f41d988cd00"

Commit message: Completed a pile more work on the various boards that comprise the project
Parts:
- H1, H2: now left out of the parts list
Changed lines of the file:
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@@
   )
   (symbol (lib_id "Mechanical:MountingHole_Pad") (at 157.48 25.4 270) (unit 1)
-    (in_bom yes) (on_board yes)
+    (in_bom no) (on_board yes)
     (property "Reference" "H2" (id 0) (at 161.29 25.4 90)
       (effects (font (size 1.27 1.27)) (justify left))
@@
   )
   (symbol (lib_id "Mechanical:MountingHole_Pad") (at 147.32 25.4 90) (unit 1)
-    (in_bom yes) (on_board yes)
+    (in_bom no) (on_board yes)
     (property "Reference" "H1" (id 0) (at 143.51 25.4 90)
       (effects (font (size 1.27 1.27)) (justify left))
