File: hardware/AudioInterface/AudioInterface.kicad_sch (KiCad schematic)
At the start: 6 parts, among them J1 I2S + SPI, J3 S/PDIF

Commit message: Completed a pile more work on the various boards that comprise the project
Parts:
- C7: value 30pF -> 30p; MFR TDK Corporation -> Yageo; MPN CGA3E2X7R1E104K080AA -> CC0603FRNPO9BN300; OC_DIGIKEY 445-5667-1-ND -> 311-3894-1-ND; OC_FARNELL 2310559 -> (none); URL_DIGIKEY https://www.digikey.com/en/products/detail/tdk-corporation/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 -> https://www.digikey.com/en/products/detail/yageo/CC0603FRNP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; URL_FARNELL https://uk.farnell.com/multicomp/mc0603b104j250ct/cap-0-1-f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 -> (none)
- H1, H2: now left out of the parts list
- J1: MFR (none) -> TE Connectivity; MPN (none) -> 1-1734592-2; OC_DIGIKEY (none) -> A100283CT-ND; URL_DIGIKEY (none) -> https://www.digikey.com/en/products/detail/te-connectivity-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
Other:
- sheet Clock Generation ports: added none; removed CSEL
- sheet Processing ports: added none; removed CSEL
