File: hardware/AudioInterface/ClockGen.kicad_sch (KiCad schematic)
At the start: 9 parts, among them U3 PLL1708, Y1 27MHz

Commit message: Completed a pile more work on the various boards that comprise the project
Parts:
- C5: MFR TDK Corporation -> muRata; MPN CGA3E2X7R1E104K080AA -> GRM188R61E106KA73D; OC_DIGIKEY 445-5667-1-ND -> 490-18214-1-ND; OC_FARNELL 2310559 -> (none); URL_DIGIKEY https://www.digikey.com/en/products/detail/tdk-corporation/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 -> https://www.digikey.com/en/products/detail/murata-electroni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; URL_FARNELL https://uk.farnell.com/multicomp/mc0603b104j250ct/cap-0-1-f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 -> (none)
Connections:
- net CSEL is gone; now on net +3V3: U3.12 (CSEL)
Other:
- note added: "CSEL held high selects SCKO1 = 12.288/24.576MHz"
Changed lines of the file:
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@@
     (stroke (width 0) (type default) (color 0 0 0 0))
   )
-  (wire (pts (xy 134.62 99.06) (xy 137.16 99.06))
+  (wire (pts (xy 121.92 99.06) (xy 137.16 99.06))
     (stroke (width 0) (type default) (color 0 0 0 0))
   )
@@
     (stroke (width 0) (type default) (color 0 0 0 0))
   )
+  (wire (pts (xy 121.92 99.06) (xy 121.92 96.52))
+    (stroke (width 0) (type default) (color 0 0 0 0))
+  )
   (wire (pts (xy 124.46 116.84) (xy 124.46 114.3))
     (stroke (width 0) (type default) (color 0 0 0 0))
@@
   (wire (pts (xy 71.12 99.06) (xy 71.12 96.52))
     (stroke (width 0) (type default) (color 0 0 0 0))
+  )
+  (text "CSEL held high selects\nSCKO1 = 12.288/24.576MHz" (at 120.65 101.6 180)
+    (effects (font (size 1.27 1.27)) (justify right bottom))
   )
   (text "Place near VCC/AGND" (at 208.28 96.52 0)
@@
   (text "Place near each VDD/DGND pair" (at 63.5 96.52 0)
     (effects (font (size 1.27 1.27)) (justify left bottom))
-  )
-  (hierarchical_label "CSEL" (shape input) (at 134.62 99.06 180)
-    (effects (font (size 1.27 1.27)) (justify right))
   )
   (hierarchical_label "SPI_CLK" (shape input) (at 134.62 93.98 180)
@@
       (effects (font (size 1.27 1.27)) hide)
     )
-    (property "Datasheet" "https://product.tdk.com/system/files/dam/doc/product/capacitor/ceramic/mlcc/catalog/mlcc_automotive_general_en.pdf" (id 3) (at 213.36 101.6 0)
-      (effects (font (size 1.27 1.27)) hide)
-    )
-    (property "OC_FARNELL" "2310559" (id 4) (at 213.36 101.6 0)
-      (effects (font (size 1.27 1.27)) hide)
-    )
-    (property "URL_FARNELL" "https://uk.farnell.com/multicomp/mc0603b104j250ct/cap-0-1-f-25v-5-x7r-0603-reel/dp/2310559" (id 5) (at 213.36 101.6 0)
-      (effects (font (size 1.27 1.27)) hide)
-    )
-    (property "MFR" "TDK Corporation" (id 6) (at 213.36 101.6 0)
-      (effects (font (size 1.27 1.27)) hide)
-    )
-    (property "MPN" "CGA3E2X7R1E104K080AA" (id 7) (at 213.36 101.6 0)
-      (effects (font (size 1.27 1.27)) hide)
-    )
-    (property "OC_DIGIKEY" "445-5667-1-ND" (id 8) (at 213.36 101.6 0)
-      (effects (font (size 1.27 1.27)) hide)
-    )
-    (property "URL_DIGIKEY" "https://www.digikey.com/en/products/detail/tdk-corporation/CGA3E2X7R1E104K080AA/2443145" (id 9) (at 213.36 101.6 0)
+    (property "Datasheet" "https://search.murata.co.jp/Ceramy/image/img/A01X/G101/ENG/GRM188R61E106KA73-01.pdf" (id 3) (at 213.36 101.6 0)
+      (effects (font (size 1.27 1.27)) hide)
+    )
+    (property "OC_FARNELL" "" (id 4) (at 213.36 101.6 0)
+      (effects (font (size 1.27 1.27)) hide)
+    )
+    (property "URL_FARNELL" "" (id 5) (at 213.36 101.6 0)
+      (effects (font (size 1.27 1.27)) hide)
+    )
+    (property "MFR" "muRata" (id 6) (at 213.36 101.6 0)
+      (effects (font (size 1.27 1.27)) hide)
+    )
+    (property "MPN" "GRM188R61E106KA73D" (id 7) (at 213.36 101.6 0)
+      (effects (font (size 1.27 1.27)) hide)
+    )
+    (property "OC_DIGIKEY" "490-18214-1-ND" (id 8) (at 213.36 101.6 0)
+      (effects (font (size 1.27 1.27)) hide)
+    )
+    (property "URL_DIGIKEY" "https://www.digikey.com/en/products/detail/murata-electronics/GRM188R61E106KA73D/9867922" (id 9) (at 213.36 101.6 0)
       (effects (font (size 1.27 1.27)) hide)
     )
@@
     (pin "2")
   )
+  (symbol (lib_id "power:+3V3") (at 121.92 96.52 0) (unit 1)
+    (in_bom yes) (on_board yes)
+    (property "Reference" "#PWR0117" (id 0) (at 121.92 100.33 0)
+      (effects (font (size 1.27 1.27)) hide)
+    )
+    (property "Value" "+3V3" (id 1) (at 121.92 92.964 0))
+    (property "Footprint" "" (id 2) (at 121.92 96.52 0)
+      (effects (font (size 1.27 1.27)) hide)
+    )
+    (property "Datasheet" "" (id 3) (at 121.92 96.52 0)
+      (effects (font (size 1.27 1.27)) hide)
+    )
+    (pin "1")
+  )
 )
