File: hardware/AudioInterface/Processing.kicad_sch (KiCad schematic)
At the start: 18 parts, among them J4 CFG, U2 ICE40HX8K-BG121, U5 GD25Q40C

Commit message: Completed a pile more work on the various boards that comprise the project
Parts:
- C23, C28: MFR (none) -> TDK; MPN (none) -> C1608X5R1C475K080AC; OC_DIGIKEY (none) -> 445-7478-1-ND; URL_DIGIKEY (none) -> https://www.digikey.com/en/products/detail/tdk-corporation/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
- C24, C25, C26, C27, C29, C30, C31, C32: MFR TDK Corporation -> Yageo; MPN CGA3E2X7R1E104K080AA -> CC0402KRX7R7BB104; OC_DIGIKEY 445-5667-1-ND -> 311-1338-1-ND; OC_FARNELL 2310559 -> (none); OC_LCSC (none) -> C60474; URL_DIGIKEY https://www.digikey.com/en/products/detail/tdk-corporation/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 -> https://www.digikey.com/en/products/detail/yageo/CC0402KRX7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; URL_FARNELL https://uk.farnell.com/multicomp/mc0603b104j250ct/cap-0-1-f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 -> (none); URL_LCSC (none) -> https://lcsc.com/product-detail/Multilayer-Ceramic-Capacito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
- D1: MFR ROHM Semiconductor -> Orient; MPN SMLEN3WBC8W1 -> ORH-W46G; OC_LCSC (none) -> C205448; URL_LCSC (none) -> https://lcsc.com/product-detail/Light-Emitting-Diodes-LED_O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
- J4: MFR (none) -> Samtec; MPN (none) -> FTSH-104-01-L-DV; OC_DIGIKEY (none) -> SAM1161-04-ND; URL_DIGIKEY (none) -> https://www.digikey.com/en/products/detail/samtec-inc/FTSH-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
- R5, R6: MFR (none) -> Vishay Dale; MPN (none) -> CRCW060310K0FKEA; OC_DIGIKEY (none) -> 541-10.0KHCT-ND; URL_DIGIKEY (none) -> https://www.digikey.com/en/products/detail/vishay-dale/CRCW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
- R8: OC_DIGIKEY (none) -> 541-6.80KHCT-ND; URL_DIGIKEY (none) -> https://www.digikey.com/en/products/detail/vishay-dale/CRCW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
- U2: MFR (none) -> Lattice Semi; MPN (none) -> ICE40HX8K-BG121; OC_DIGIKEY (none) -> 220-2148-ND; URL_DIGIKEY (none) -> https://www.digikey.com/en/products/detail/lattice-semicond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
Connections:
- net CSEL: no longer names the net of U2.A4 (IOT_211)
- no-connect marks 67 -> 68
