File: hardware/AudioInterface/USB.kicad_sch (KiCad schematic)
At the start: 14 parts, among them J2 USB_C_Receptacle_USB2.0, U1 USB3318, U4 SP3400-02UTG, X1 13MHz

Commit message: Completed a pile more work on the various boards that comprise the project
Parts:
- C22: MFR (none) -> TDK; MPN (none) -> C1608X5R1C475K080AC; OC_DIGIKEY (none) -> 445-7478-1-ND; URL_DIGIKEY (none) -> https://www.digikey.com/en/products/detail/tdk-corporation/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
- J2: MFR (none) -> Korean Hroparts; MPN (none) -> TYPE-C-31-M-12; OC_LCSC (none) -> C165948; URL_LCSC (none) -> https://lcsc.com/product-detail/USB-Connectors_Korean-Hropa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
- R1: MFR (none) -> Vishay Dale; MPN (none) -> CRCW06031M00FKEA; OC_DIGIKEY (none) -> 541-1.00MHCT-ND; URL_DIGIKEY (none) -> https://www.digikey.com/en/products/detail/vishay-dale/CRCW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
- R2, R3: MFR (none) -> Vishay Dale; MPN (none) -> CRCW06035K10FKEA; OC_DIGIKEY (none) -> 541-5.10KHCT-ND; URL_DIGIKEY (none) -> https://www.digikey.com/en/products/detail/vishay-dale/CRCW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
- R4: MFR (none) -> Vishay Dale; MPN (none) -> CRCW06038K06FKEA; OC_DIGIKEY (none) -> 541-8.06KHCT-ND; URL_DIGIKEY (none) -> https://www.digikey.com/en/products/detail/vishay-dale/CRCW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
- R7: MFR (none) -> Vishay Dale; MPN (none) -> CRCW060310K0FKEA; OC_DIGIKEY (none) -> 541-10.0KHCT-ND; URL_DIGIKEY (none) -> https://www.digikey.com/en/products/detail/vishay-dale/CRCW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
- U1: OC_DIGIKEY (none) -> 638-1064-1-ND; URL_DIGIKEY (none) -> https://www.digikey.com/en/products/detail/microchip-techno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
Changed lines of the file:
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@@
       (effects (font (size 1.27 1.27)) hide)
     )
-    (property "Datasheet" "https://www.usb.org/sites/default/files/documents/usb_type-c.zip" (id 3) (at 118.11 104.14 0)
+    (property "Datasheet" "https://datasheet.lcsc.com/lcsc/2108131730_Korean-Hroparts-Elec-TYPE-C-31-M-12_C165948.pdf" (id 3) (at 118.11 104.14 0)
+      (effects (font (size 1.27 1.27)) hide)
+    )
+    (property "MFR" "Korean Hroparts" (id 4) (at 114.3 101.6 0)
+      (effects (font (size 1.27 1.27)) hide)
+    )
+    (property "MPN" "TYPE-C-31-M-12" (id 5) (at 114.3 101.6 0)
+      (effects (font (size 1.27 1.27)) hide)
+    )
+    (property "OC_LCSC" "C165948" (id 6) (at 114.3 101.6 0)
+      (effects (font (size 1.27 1.27)) hide)
+    )
+    (property "URL_LCSC" "https://lcsc.com/product-detail/USB-Connectors_Korean-Hroparts-Elec-TYPE-C-31-M-12_C165948.html" (id 7) (at 114.3 101.6 0)
       (effects (font (size 1.27 1.27)) hide)
     )
@@
       (effects (font (size 1.27 1.27)) hide)
     )
-    (property "Datasheet" "" (id 3) (at 233.68 71.12 0)
-      (effects (font (size 1.27 1.27)) hide)
-    )
-    (property "MFR" "" (id 6) (at 233.68 71.12 0)
-      (effects (font (size 1.27 1.27)) hide)
-    )
-    (property "MPN" "" (id 7) (at 233.68 71.12 0)
+    (property "Datasheet" "https://product.tdk.com/system/files/dam/doc/product/capacitor/ceramic/mlcc/charasheet/c1608x5r1c475k080ac.pdf" (id 3) (at 233.68 71.12 0)
+      (effects (font (size 1.27 1.27)) hide)
+    )
+    (property "MFR" "TDK" (id 6) (at 233.68 71.12 0)
+      (effects (font (size 1.27 1.27)) hide)
+    )
+    (property "MPN" "C1608X5R1C475K080AC" (id 7) (at 233.68 71.12 0)
       (effects (font (size 0 0)) hide)
     )
-    (property "OC_DIGIKEY" "" (id 8) (at 233.68 71.12 0)
-      (effects (font (size 1.27 1.27)) hide)
-    )
-    (property "URL_DIGIKEY" "" (id 9) (at 233.68 71.12 0)
+    (property "OC_DIGIKEY" "445-7478-1-ND" (id 8) (at 233.68 71.12 0)
+      (effects (font (size 1.27 1.27)) hide)
+    )
+    (property "URL_DIGIKEY" "https://www.digikey.com/en/products/detail/tdk-corporation/C1608X5R1C475K080AC/2732913" (id 9) (at 233.68 71.12 0)
       (effects (font (size 1.27 1.27)) hide)
     )
@@
       (effects (font (size 1.27 1.27)) hide)
     )
-    (property "Datasheet" "~" (id 3) (at 132.08 96.52 0)
+    (property "Datasheet" "https://www.vishay.com/docs/20035/dcrcwe3.pdf" (id 3) (at 132.08 96.52 0)
+      (effects (font (size 1.27 1.27)) hide)
+    )
+    (property "MFR" "Vishay Dale" (id 4) (at 132.08 96.52 0)
+      (effects (font (size 1.27 1.27)) hide)
+    )
+    (property "MPN" "CRCW06035K10FKEA" (id 5) (at 132.08 96.52 0)
+      (effects (font (size 1.27 1.27)) hide)
+    )
+    (property "OC_DIGIKEY" "541-5.10KHCT-ND" (id 6) (at 132.08 96.52 0)
+      (effects (font (size 1.27 1.27)) hide)
+    )
+    (property "URL_DIGIKEY" "https://www.digikey.com/en/products/detail/vishay-dale/CRCW06035K10FKEA/1174748" (id 7) (at 132.08 96.52 0)
       (effects (font (size 1.27 1.27)) hide)
     )
@@
     )
     (property "MPN" "USB3318-CP-TR" (id 5) (at 177.8 124.46 0)
+      (effects (font (size 1.27 1.27)) hide)
+    )
+    (property "OC_DIGIKEY" "638-1064-1-ND" (id 6) (at 177.8 91.44 0)
+      (effects (font (size 1.27 1.27)) hide)
+    )
+    (property "URL_DIGIKEY" "https://www.digikey.com/en/products/detail/microchip-technology/USB3318-CP-TR/1825071" (id 7) (at 177.8 91.44 0)
       (effects (font (size 1.27 1.27)) hide)
     )
@@
       (effects (font (size 1.27 1.27)) hide)
     )
-    (property "Datasheet" "~" (id 3) (at 114.3 132.08 0)
+    (property "Datasheet" "https://www.vishay.com/docs/20035/dcrcwe3.pdf" (id 3) (at 114.3 132.08 0)
+      (effects (font (size 1.27 1.27)) hide)
+    )
+    (property "MFR" "Vishay Dale" (id 4) (at 114.3 132.08 0)
+      (effects (font (size 1.27 1.27)) hide)
+    )
+    (property "MPN" "CRCW06031M00FKEA" (id 5) (at 114.3 132.08 0)
+      (effects (font (size 1.27 1.27)) hide)
+    )
+    (property "OC_DIGIKEY" "541-1.00MHCT-ND" (id 6) (at 114.3 132.08 0)
+      (effects (font (size 1.27 1.27)) hide)
+    )
+    (property "URL_DIGIKEY" "https://www.digikey.com/en/products/detail/vishay-dale/CRCW06031M00FKEA/1175010" (id 7) (at 114.3 132.08 0)
       (effects (font (size 1.27 1.27)) hide)
     )
@@
       (effects (font (size 1.27 1.27)) hide)
     )
-    (property "Datasheet" "~" (id 3) (at 157.48 81.28 0)
+    (property "Datasheet" "https://www.vishay.com/docs/20035/dcrcwe3.pdf" (id 3) (at 157.48 81.28 0)
+      (effects (font (size 1.27 1.27)) hide)
+    )
+    (property "MFR" "Vishay Dale" (id 4) (at 157.48 81.28 0)
+      (effects (font (size 1.27 1.27)) hide)
+    )
+    (property "MPN" "CRCW06038K06FKEA" (id 5) (at 157.48 81.28 0)
+      (effects (font (size 1.27 1.27)) hide)
+    )
+    (property "OC_DIGIKEY" "541-8.06KHCT-ND" (id 6) (at 157.48 81.28 0)
+      (effects (font (size 1.27 1.27)) hide)
+    )
+    (property "URL_DIGIKEY" "https://www.digikey.com/en/products/detail/vishay-dale/CRCW06038K06FKEA/1174771" (id 7) (at 157.48 81.28 0)
       (effects (font (size 1.27 1.27)) hide)
     )
@@
       (effects (font (size 1.27 1.27)) hide)
     )
-    (property "Datasheet" "~" (id 3) (at 132.08 93.98 0)
+    (property "Datasheet" "https://www.vishay.com/docs/20035/dcrcwe3.pdf" (id 3) (at 132.08 93.98 0)
+      (effects (font (size 1.27 1.27)) hide)
+    )
+    (property "MFR" "Vishay Dale" (id 4) (at 132.08 93.98 0)
+      (effects (font (size 1.27 1.27)) hide)
+    )
+    (property "MPN" "CRCW06035K10FKEA" (id 5) (at 132.08 93.98 0)
+      (effects (font (size 1.27 1.27)) hide)
+    )
+    (property "OC_DIGIKEY" "541-5.10KHCT-ND" (id 6) (at 132.08 93.98 0)
+      (effects (font (size 1.27 1.27)) hide)
+    )
+    (property "URL_DIGIKEY" "https://www.digikey.com/en/products/detail/vishay-dale/CRCW06035K10FKEA/1174748" (id 7) (at 132.08 93.98 0)
       (effects (font (size 1.27 1.27)) hide)
     )
@@
       (effects (font (size 1.27 1.27)) hide)
     )
-    (property "Datasheet" "~" (id 3) (at 157.48 99.06 0)
-      (effects (font (size 1.27 1.27)) hide)
-    )
+    (property "Datasheet" "https://www.vishay.com/docs/20035/dcrcwe3.pdf" (id 3) (at 157.48 99.06 0)
+      (effects (font (size 1.27 1.27)) hide)
+    )
+    (property "MFR" "Vishay Dale" (id 4) (at 157.48 99.06 0)
+      (effects (font (size 1.27 1.27)) hide)
+    )
+    (property "MPN" "CRCW060310K0FKEA" (id 5) (at 157.48 99.06 0)
+      (effects (font (size 1.27 1.27)) hide)
+    )
+    (property "OC_DIGIKEY" "541-10.0KHCT-ND" (id 6) (at 157.48 99.06 0)
+      (effects (font (size 1.27 1.27)) hide)
+    )
+    (property "URL_DIGIKEY" "https://www.digikey.com/en/products/detail/vishay-dale/CRCW060310K0FKEA/1174782" (id 7) (at 157.48 99.06 0)
+      (effects (font (size 1.27 1.27)) hide)
+    )
