File: hardware/SignalRouter/SignalRouter.kicad_sch (KiCad schematic)
At the start: 28 parts, among them J1 Src Control, J2 EXT_R, J3 EXT_L, J4 INT_R, J5 INT_L, J6 Preamp, K1 EC2-12TNU, Q1 DMN65D8L, Q10 DMN65D8L, Q2 DMN65D8L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

Commit message: Completed a pile more work on the various boards that comprise the project
Parts:
- H1, H2: now left out of the parts list
Changed lines of the file:
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@@
   )
   (symbol (lib_id "Mechanical:MountingHole_Pad") (at 228.6 45.72 0) (unit 1)
-    (in_bom yes) (on_board yes)
+    (in_bom no) (on_board yes)
     (property "Reference" "H1" (id 0) (at 228.6 39.37 0))
     (property "Value" "MountingHole_Pad" (id 1) (at 228.6 41.275 0))
@@
   )
   (symbol (lib_id "Mechanical:MountingHole_Pad") (at 254 45.72 0) (unit 1)
-    (in_bom yes) (on_board yes)
+    (in_bom no) (on_board yes)
     (property "Reference" "H2" (id 0) (at 254 39.37 0))
     (property "Value" "MountingHole_Pad" (id 1) (at 254 41.275 0))
